File: DigitalClock/min_counter.kicad_sch (KiCad schematic)
At the start: 2 parts

Commit message: added minute counter schematic"
Parts:
- added U? (x10): 74LS86, symbol 74xx:74LS86
- added U? (x15): 74LS74, symbol 74xx:74LS74
- added U? (x25): 74LS08, symbol 74xx:74LS08
Connections:
- net CLK_1min: now also U?.11 (C), U?.11 (C), U?.11 (C), U?.3 (C), U?.3 (C), U?.3 (C)
- net min_ones_0: now also U?.1, U?.1, U?.1, U?.5 (Q)
- net min_ones_1: now also U?.2, U?.2, U?.9 (Q)
- net min_ones_2: now also U?.5, U?.5, U?.5 (Q)
- net min_ones_3: now also U?.10, U?.5, U?.9 (Q)
- net min_tens_0: now also U?.1, U?.1, U?.5 (Q), U?.9
- net min_tens_1: now also U?.10, U?.2, U?.9 (Q)
- net min_tens_2: now also U?.13, U?.5, U?.5 (Q), U?.9
- net min_tens_3: now also U?.10, U?.9 (Q)
- net ~{RESET_PULSE}: now also U?.1 (~{R}), U?.1 (~{R}), U?.1 (~{R}), U?.1 (~{R}), U?.13 (~{R}), U?.13 (~{R}), U?.13 (~{R}), U?.13 (~{R})
- net =9?: now reaches U?.3
- net =9?: now also U?.13, U?.2 (D), U?.8
- net ~{=9?}: now reaches U?.4
- net ~{=9?}: now also U?.10, U?.13, U?.2, U?.5
- net =59?: now reaches U?.5
- net =59?: now also U?.11, U?.12 (D)
- net ~{=59?}: now reaches U?.6
- net ~{=59?}: now also U?.10, U?.13, U?.2, U?.5
- new net: U?.6, U?.9 (x2)
- new net: U?.12, U?.6
- new net: U?.12, U?.8 (x2)
- new net: U?.3, U?.4 (x3)
- new net: U?.3, U?.9
- new net: U?.5, U?.8
- new net: U?.10, U?.6
- new net +5V: U?.1 (~{R}), U?.10 (~{S}), U?.10 (~{S}), U?.10 (~{S}), U?.10 (~{S}), U?.10 (~{S}), U?.13 (~{R}), U?.14 (VCC), U?.14 (VCC), U?.14 (VCC), U?.14 (VCC), U?.14 (VCC), U?.14 (VCC), U?.14 (VCC), U?.14 (VCC), U?.14 (VCC), U?.14 (VCC), U?.14 (VCC), U?.14 (VCC), U?.4 (~{S}), U?.4 (~{S}), U?.4 (~{S}), U?.4 (~{S}), U?.4 (~{S})
- new net CLK_10min: U?.11 (C), U?.11 (C), U?.3 (C), U?.3 (C), U?.5 (Q)
- new net CLK_1hour: U?.9 (Q)
- new net GND: U?.12, U?.12, U?.12, U?.13, U?.13, U?.13, U?.7 (GND), U?.7 (GND), U?.7 (GND), U?.7 (GND), U?.7 (GND), U?.7 (GND), U?.7 (GND), U?.7 (GND), U?.7 (GND), U?.7 (GND), U?.7 (GND), U?.7 (GND)
- new net ones_D0: U?.2 (D), U?.3
- new net ones_D1: U?.12 (D), U?.6
- new net ones_D2: U?.2 (D), U?.8
- new net ones_D3: U?.11, U?.12 (D)
- new net ones_Q01: U?.3, U?.4, U?.4
- new net ones_Q012: U?.6, U?.9
- new net tens_D0: U?.2 (D), U?.3
- new net tens_D1: U?.12 (D), U?.6
- new net tens_D2: U?.2 (D), U?.8
- new net tens_D3: U?.11, U?.12 (D)
- new net tens_Q01: U?.12, U?.4, U?.8
- new net tens_Q012: U?.11, U?.9
- new net ~{ones_Q0}: U?.1, U?.6 (~{Q})
- new net ~{ones_Q1}: U?.2, U?.8 (~{Q})
- new net ~{ones_Q2}: U?.4, U?.6 (~{Q})
- new net ~{ones_Q3}: U?.8 (~{Q})
- new net ~{tens_Q0}: U?.1, U?.6 (~{Q})
- new net ~{tens_Q1}: U?.2, U?.8 (~{Q})
- new net ~{tens_Q2}: U?.6 (~{Q})
- new net ~{tens_Q3}: U?.10, U?.8 (~{Q})
Other:
- moved on the sheet: U?B, U?C

Commit message: finished kicad schematic
Parts:
- gave numbers to parts that had none: 13
Connections:
- no-connect marks 0 -> 5

Commit message: about to begin layout
Parts:
- U15, U26, U27, U28, U29, U30, U31, U32, U33, U34, U35, U36, U37: footprint (none) -> Package_DIP:DIP-14_W7.62mm

Commit message: started routing
Connections:
- net GND: now also U28.12, U28.13; no longer U37.12, U37.13
- net min_ones_0: now also U33.1; no longer U29.1
- net min_ones_1: now also U33.2; no longer U29.2
- net min_ones_2: now also U33.5; no longer U29.5
- net min_tens_0: now also U29.1; no longer U33.1
- net min_tens_2: now also U29.9, U33.13; no longer U32.13, U32.9
- net ones_D2: now also U32.8; no longer U29.8
- net ones_D3: now also U32.11; no longer U28.11
- net ones_Q01: now also U33.3, U33.4; no longer U29.3, U29.4
- net ones_Q012: now also U33.6; no longer U29.6
- net tens_D3: now also U37.11; no longer U33.11
- net tens_Q01: now also U33.12; no longer U32.12
- net tens_Q012: now also U33.11; no longer U32.11
- net ~{=59?}: now also U37.13; no longer U33.13
- net ~{=9?}: now also U32.10, U32.13; no longer U28.13, U29.10
- net ~{tens_Q1}: now also U29.2; no longer U33.2
- net ~{tens_Q3}: now also U29.10; no longer U32.10
- net at U30.6: now also U32.9; no longer U29.9
- net at U29.12: now also U29.6; no longer U33.6
- net at U30.8: now also U32.12; no longer U28.12
- net at U36.8: now also U37.12; no longer U33.12
- new net: U29.5, U29.8
- new net: U29.3, U29.4
Other:
- moved on the sheet: U28D, U29A, U29B, U29C, U32C, U32D, U33A, U33B, U33D, U37D
