File: DigitalClock/DigitalClock.kicad_pcb (KiCad board)
At the start: 2 copper layers, 203.2 x 101.6 mm, 84 parts, among them J1 Battery, Q1 2N3904, Q2 2N3904, Q3 2N3904, SW1 +HOUR, SW2 SET TIME, SW3 +MIN, U1 74LS47, U10 HDSP-7801, U11 LM1117-5.0, U12 74LS47, U13 74LS74, U14 HDSP-7801, U15 74LS04, U16 74LS08, U17 74LS74, U18 74LS86, U19 74LS86, U2 NE555P, U20 74LS08, U21 74LS08, U22 74LS74, U23 74LS74, U24 74LS74, U25 74LS08, U26 74LS74, U27 74LS74, U28 74LS08, U29 74LS08, U3 HDSP-7801, U30 74LS86, U31 74LS74, U32 74LS08, U33 74LS08, U34 74LS74, U35 74LS74, U36 74LS86, U37 74LS08, U38 74LS74, U39 74LS86, U4 74LS08, U40 74LS74, U41 74LS74, U42 74LS08, U43 74LS08, U44 74LS86, U45 74LS74, U46 74LS74, U47 74LS08, U48 74LS08, U49 74LS32, U5 74LS32, U50 74LS32, U51 74LS08, U52 74LS32, U53 74LS08, U6 74LS47, U7 HDSP-7801, U8 74LS47, U9 74LS74

Commit message: more routing
Parts:
- added R16: 1k, Resistor_THT:R_Axial_DIN0207_L6.3mm_D2.5mm_P10.16mm_Horizontal, F.Cu at (365.5, 69.4)
- added R17: 1k, Resistor_THT:R_Axial_DIN0207_L6.3mm_D2.5mm_P10.16mm_Horizontal, F.Cu at (352.2, 73.4)
- added R18: 1k, Resistor_THT:R_Axial_DIN0207_L6.3mm_D2.5mm_P10.16mm_Horizontal, F.Cu at (365.5, 65.3)
- added R19: 1k, Resistor_THT:R_Axial_DIN0207_L6.3mm_D2.5mm_P10.16mm_Horizontal, F.Cu at (352.2, 77.5)
- added R20: 1k, Resistor_THT:R_Axial_DIN0207_L6.3mm_D2.5mm_P10.16mm_Horizontal, F.Cu at (338.9, 89.6)
- added R21: 1k, Resistor_THT:R_Axial_DIN0207_L6.3mm_D2.5mm_P10.16mm_Horizontal, F.Cu at (352.2, 89.6)
- added R22: 1k, Resistor_THT:R_Axial_DIN0207_L6.3mm_D2.5mm_P10.16mm_Horizontal, F.Cu at (325.6, 73.4)
- added R23: 1k, Resistor_THT:R_Axial_DIN0207_L6.3mm_D2.5mm_P10.16mm_Horizontal, F.Cu at (325.6, 81.5)
- added R24: 1k, Resistor_THT:R_Axial_DIN0207_L6.3mm_D2.5mm_P10.16mm_Horizontal, F.Cu at (365.5, 77.5)
- added R25: 1k, Resistor_THT:R_Axial_DIN0207_L6.3mm_D2.5mm_P10.16mm_Horizontal, F.Cu at (338.9, 73.4)
- added R26: 1k, Resistor_THT:R_Axial_DIN0207_L6.3mm_D2.5mm_P10.16mm_Horizontal, F.Cu at (352.2, 69.4)
- added R27: 1k, Resistor_THT:R_Axial_DIN0207_L6.3mm_D2.5mm_P10.16mm_Horizontal, F.Cu at (325.6, 89.6)
- added R28: 1k, Resistor_THT:R_Axial_DIN0207_L6.3mm_D2.5mm_P10.16mm_Horizontal, F.Cu at (338.9, 77.5)
- added R29: 1k, Resistor_THT:R_Axial_DIN0207_L6.3mm_D2.5mm_P10.16mm_Horizontal, F.Cu at (325.6, 85.6)
- added R30: 1k, Resistor_THT:R_Axial_DIN0207_L6.3mm_D2.5mm_P10.16mm_Horizontal, F.Cu at (338.9, 69.4)
- added R31: 1k, Resistor_THT:R_Axial_DIN0207_L6.3mm_D2.5mm_P10.16mm_Horizontal, F.Cu at (338.9, 93.7)
- added R32: 1k, Resistor_THT:R_Axial_DIN0207_L6.3mm_D2.5mm_P10.16mm_Horizontal, F.Cu at (325.6, 93.7)
- added R33: 1k, Resistor_THT:R_Axial_DIN0207_L6.3mm_D2.5mm_P10.16mm_Horizontal, F.Cu at (325.6, 77.5)
- added R34: 1k, Resistor_THT:R_Axial_DIN0207_L6.3mm_D2.5mm_P10.16mm_Horizontal, F.Cu at (365.5, 81.5)
- added R35: 1k, Resistor_THT:R_Axial_DIN0207_L6.3mm_D2.5mm_P10.16mm_Horizontal, F.Cu at (338.9, 81.5)
- added R36: 1k, Resistor_THT:R_Axial_DIN0207_L6.3mm_D2.5mm_P10.16mm_Horizontal, F.Cu at (338.9, 65.3)
- added R37: 1k, Resistor_THT:R_Axial_DIN0207_L6.3mm_D2.5mm_P10.16mm_Horizontal, F.Cu at (338.9, 85.6)
- added R38: 1k, Resistor_THT:R_Axial_DIN0207_L6.3mm_D2.5mm_P10.16mm_Horizontal, F.Cu at (352.2, 65.3)
- added R39: 1k, Resistor_THT:R_Axial_DIN0207_L6.3mm_D2.5mm_P10.16mm_Horizontal, F.Cu at (365.5, 73.4)
- added R40: 1k, Resistor_THT:R_Axial_DIN0207_L6.3mm_D2.5mm_P10.16mm_Horizontal, F.Cu at (352.2, 81.5)
- added R41: 1k, Resistor_THT:R_Axial_DIN0207_L6.3mm_D2.5mm_P10.16mm_Horizontal, F.Cu at (325.6, 69.4)
- added R42: 1k, Resistor_THT:R_Axial_DIN0207_L6.3mm_D2.5mm_P10.16mm_Horizontal, F.Cu at (352.2, 85.6)
- added R43: 1k, Resistor_THT:R_Axial_DIN0207_L6.3mm_D2.5mm_P10.16mm_Horizontal, F.Cu at (325.6, 65.3)
- moved U8 323.9 mm to (351.0, 40.6)
- moved U1 312.2 mm to (329.4, 40.6)
- moved U6 302.3 mm to (340.3, 40.5)
- moved U12 281.3 mm to (361.5, 40.6)
- moved U14 247.0 mm to (263.2, 117.1), turned to 90 degrees
- moved U9 234.4 mm to (248.5, -21.4)
- moved U7 223.5 mm to (234.5, 117.1), turned to 90 degrees
- moved U10 222.1 mm to (248.9, 117.1), turned to 90 degrees
- moved D2 217.9 mm to (271.2, 96.2)
- moved U3 187.7 mm to (220.1, 117.1), turned to 90 degrees
- moved U38 183.1 mm to (233.7, 21.5)
- moved U39 183.1 mm to (190.3, 40.9)
- moved U40 183.1 mm to (255.4, 21.5)
- moved U41 183.1 mm to (266.3, 21.5)
- moved U42 183.1 mm to (201.2, 40.9)
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Connections:
- U1 pad 10: Net-(U1-Pad10) -> Net-(R19-Pad1)
- U1 pad 11: Net-(U1-Pad11) -> Net-(R18-Pad1)
- U1 pad 12: Net-(U1-Pad12) -> Net-(R17-Pad1)
- U1 pad 13: Net-(U1-Pad13) -> Net-(R16-Pad1)
- U1 pad 14: Net-(U1-Pad14) -> Net-(R22-Pad1)
- U1 pad 15: Net-(U1-Pad15) -> Net-(R21-Pad1)
- U1 pad 9: Net-(U1-Pad9) -> Net-(R20-Pad1)
- U10 pad 10: Net-(U10-Pad10) -> Net-(R30-Pad2)
- U10 pad 2: Net-(U10-Pad2) -> Net-(R35-Pad2)
- U10 pad 3: Net-(U10-Pad3) -> Net-(R36-Pad2)
- U10 pad 4: Net-(U10-Pad4) -> Net-(R34-Pad2)
- U10 pad 5: Net-(U10-Pad5) -> Net-(R33-Pad2)
- U10 pad 8: Net-(U10-Pad8) -> Net-(R32-Pad2)
- U10 pad 9: Net-(U10-Pad9) -> Net-(R31-Pad2)
- U12 pad 10: Net-(U12-Pad10) -> Net-(R40-Pad1)
- U12 pad 11: Net-(U12-Pad11) -> Net-(R39-Pad1)
- U12 pad 12: Net-(U12-Pad12) -> Net-(R38-Pad1)
- U12 pad 13: Net-(U12-Pad13) -> Net-(R37-Pad1)
- U12 pad 14: Net-(U12-Pad14) -> Net-(R43-Pad1)
- U12 pad 15: Net-(U12-Pad15) -> Net-(R42-Pad1)
- U12 pad 9: Net-(U12-Pad9) -> Net-(R41-Pad1)
- U14 pad 10: Net-(U12-Pad13) -> Net-(R37-Pad2)
- U14 pad 2: Net-(U12-Pad15) -> Net-(R42-Pad2)
- U14 pad 3: Net-(U12-Pad14) -> Net-(R43-Pad2)
- U14 pad 4: Net-(U12-Pad9) -> Net-(R41-Pad2)
- U14 pad 5: Net-(U12-Pad10) -> Net-(R40-Pad2)
- U14 pad 8: Net-(U12-Pad11) -> Net-(R39-Pad2)
- U14 pad 9: Net-(U12-Pad12) -> Net-(R38-Pad2)
- U23 pad 11: /CLK_1sec -> GND
- U23 pad 12: /sec_counter/D5 -> GND
- U23 pad 13: /~{RESET_PULSE} -> +5V
- U23 pad 8: /sec_counter/~{Q5} -> unconnected-(U23-Pad8)
- U23 pad 9: /sec_counter/Q5 -> unconnected-(U23-Pad9)
- U24 pad 11: GND -> /CLK_1sec
- U24 pad 12: GND -> /sec_counter/D5
- U24 pad 13: +5V -> /~{RESET_PULSE}
- U24 pad 8: unconnected-(U24-Pad8) -> /sec_counter/~{Q5}
- U24 pad 9: unconnected-(U24-Pad9) -> /sec_counter/Q5
- U3 pad 10: Net-(U1-Pad13) -> Net-(R16-Pad2)
- U3 pad 2: Net-(U1-Pad15) -> Net-(R21-Pad2)
- U3 pad 3: Net-(U1-Pad14) -> Net-(R22-Pad2)
- U3 pad 4: Net-(U1-Pad9) -> Net-(R20-Pad2)
- U3 pad 5: Net-(U1-Pad10) -> Net-(R19-Pad2)
- U3 pad 8: Net-(U1-Pad11) -> Net-(R18-Pad2)
- U3 pad 9: Net-(U1-Pad12) -> Net-(R17-Pad2)
- U6 pad 10: Net-(U6-Pad10) -> Net-(R26-Pad1)
- U6 pad 11: Net-(U6-Pad11) -> Net-(R25-Pad1)
- U6 pad 12: Net-(U6-Pad12) -> Net-(R24-Pad1)
- U6 pad 13: Net-(U6-Pad13) -> Net-(R23-Pad1)
- U6 pad 14: Net-(U6-Pad14) -> Net-(R29-Pad1)
- U6 pad 15: Net-(U6-Pad15) -> Net-(R28-Pad1)
- U6 pad 9: Net-(U6-Pad9) -> Net-(R27-Pad1)
- U7 pad 10: Net-(U6-Pad13) -> Net-(R23-Pad2)
- U7 pad 2: Net-(U6-Pad15) -> Net-(R28-Pad2)
- U7 pad 3: Net-(U6-Pad14) -> Net-(R29-Pad2)
- U7 pad 4: Net-(U6-Pad9) -> Net-(R27-Pad2)
- U7 pad 5: Net-(U6-Pad10) -> Net-(R26-Pad2)
- U7 pad 8: Net-(U6-Pad11) -> Net-(R25-Pad2)
- U7 pad 9: Net-(U6-Pad12) -> Net-(R24-Pad2)
- U8 pad 10: Net-(U10-Pad5) -> Net-(R33-Pad1)
- U8 pad 11: Net-(U10-Pad8) -> Net-(R32-Pad1)
- U8 pad 12: Net-(U10-Pad9) -> Net-(R31-Pad1)
- U8 pad 13: Net-(U10-Pad10) -> Net-(R30-Pad1)
- U8 pad 14: Net-(U10-Pad3) -> Net-(R36-Pad1)
- U8 pad 15: Net-(U10-Pad2) -> Net-(R35-Pad1)
- U8 pad 9: Net-(U10-Pad4) -> Net-(R34-Pad1)
Other:
- board text added: "PM"
- board text added: "SET TIME"

Commit message: more layout
Parts:
- added U54: 74LS04, Package_DIP:DIP-14_W7.62mm, F.Cu at (144.0, 106.7)
- SW1: value +HOUR -> SW_Push; footprint Button_Switch_THT:Push_E-Switch_KS01Q01 -> Button_Switch_THT:SW_PUSH_6mm
- SW2: value SET TIME -> SW_Push; footprint Button_Switch_THT:Push_E-Switch_KS01Q01 -> Button_Switch_THT:SW_PUSH_6mm
- SW3: value +MIN -> SW_Push; footprint Button_Switch_THT:Push_E-Switch_KS01Q01 -> Button_Switch_THT:SW_PUSH_6mm
- moved R14 225.6 mm to (99.6, 105.5)
- moved Q3 214.7 mm to (106.6, 100.7)
- moved Q2 208.6 mm to (99.9, 100.7)
- moved C5 195.2 mm to (93.4, 107.3), turned to 180 degrees
- moved R15 194.8 mm to (273.1, 109.2), turned to 90 degrees
- moved U9 186.0 mm to (113.7, 106.7), turned to 90 degrees
- moved R2 185.2 mm to (166.9, 110.5), turned to 180 degrees
- moved R7 181.0 mm to (143.5, 110.5)
- moved R1 177.1 mm to (166.9, 114.2), turned to 180 degrees
- moved R13 176.6 mm to (185.9, 112.3), turned to 90 degrees
- moved R18 174.7 mm to (191.4, 78.5), turned to -90 degrees
- moved R8 169.3 mm to (153.7, 114.2), turned to 180 degrees
- moved R11 168.7 mm to (99.6, 109.3)
- moved R16 167.8 mm to (198.0, 78.5), turned to -90 degrees
- moved C1 167.7 mm to (106.9, 118.2), turned to 90 degrees
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Connections:
- net /+HOUR renamed Net-(C2-Pad1)
- net /+MIN renamed Net-(C4-Pad1)
- C3 pad 1: /RESET_BUTTON -> Net-(C3-Pad1)
- R1 pad 1: Net-(R1-Pad1) -> Net-(R4-Pad1)
- R1 pad 2: GND -> +5V
- R2 pad 2: GND -> +5V
- R3 pad 1: Net-(R3-Pad1) -> Net-(R6-Pad1)
- R3 pad 2: GND -> +5V
- R4 pad 1: Net-(R1-Pad1) -> Net-(R4-Pad1)
- R5 pad 2: /RESET_BUTTON -> Net-(C3-Pad1)
- R6 pad 1: Net-(R3-Pad1) -> Net-(R6-Pad1)
- SW1 pad 1: +5V -> GND
- SW1 pad 2: Net-(R1-Pad1) -> unconnected-(SW1-Pad2)
- SW2 pad 1: +5V -> GND
- SW3 pad 1: +5V -> GND
- SW3 pad 2: Net-(R3-Pad1) -> Net-(R6-Pad1)
Other:
- board text removed: "PM"
- board text removed: "SET TIME"

Commit message: started routing
Parts:
- moved U44 84.1 mm to (185.3, 22.3)
- moved U41 83.9 mm to (185.3, 44.1)
- moved U46 83.7 mm to (266.2, 44.1)
- moved U31 61.9 mm to (115.3, 90.9), turned to 90 degrees
- moved U20 58.0 mm to (100.6, 79.0)
- moved U22 57.9 mm to (88.0, 22.3)
- moved U24 56.5 mm to (100.6, 22.3), turned to 0 degrees
- moved U32 56.0 mm to (115.2, 78.5), turned to 90 degrees
- moved U36 54.7 mm to (115.3, 22.4)
- moved U50 51.6 mm to (208.2, 22.3)
- moved U30 46.8 mm to (115.5, 44.1), turned to 0 degrees
- moved U51 46.3 mm to (254.6, 22.1)
- moved U18 42.8 mm to (75.7, 44.1)
- moved U19 42.2 mm to (75.8, 79.0)
- moved U42 41.2 mm to (231.2, 22.2)
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Connections:
- R1 pad 1: Net-(R4-Pad1) -> Net-(R1-Pad1)
- R4 pad 1: Net-(R4-Pad1) -> Net-(R1-Pad1)
- SW1 pad 2: unconnected-(SW1-Pad2) -> Net-(R1-Pad1)
- U18 pad 1: /sec_counter/Q01234 -> /sec_counter/Q0
- U18 pad 2: /sec_counter/Q5 -> /sec_counter/Q1
- U19 pad 1: /sec_counter/Q0 -> /sec_counter/Q01234
- U19 pad 2: /sec_counter/Q1 -> /sec_counter/Q5
- U20 pad 1: Net-(U16-Pad11) -> /sec_counter/~{=59?}
- U20 pad 10: Net-(U18-Pad6) -> Net-(U18-Pad8)
- U20 pad 11: /sec_counter/D3 -> /sec_counter/D4
- U20 pad 13: Net-(U18-Pad8) -> Net-(U18-Pad11)
- U20 pad 2: Net-(U16-Pad8) -> Net-(U18-Pad3)
- U20 pad 3: /sec_counter/=59? -> /sec_counter/D1
- U20 pad 5: Net-(U18-Pad3) -> Net-(U18-Pad6)
- U20 pad 6: /sec_counter/D5 -> /sec_counter/D2
- U20 pad 8: /sec_counter/D2 -> /sec_counter/D3
- U21 pad 10: /sec_counter/Q3 -> GND
- U21 pad 11: /sec_counter/Q01234 -> unconnected-(U21-Pad11)
- U21 pad 12: /sec_counter/Q0123 -> GND
- U21 pad 13: /sec_counter/Q4 -> GND
- U21 pad 2: Net-(U18-Pad11) -> Net-(U19-Pad3)
- U21 pad 3: /sec_counter/D4 -> /sec_counter/D5
- U21 pad 4: /sec_counter/~{=59?} -> Net-(U16-Pad11)
- U21 pad 5: Net-(U19-Pad3) -> Net-(U16-Pad8)
- U21 pad 6: /sec_counter/D1 -> /sec_counter/=59?
- U21 pad 8: /sec_counter/Q0123 -> unconnected-(U21-Pad8)
- U21 pad 9: /sec_counter/Q012 -> GND
- U25 pad 10: GND -> /sec_counter/Q3
- U25 pad 11: unconnected-(U25-Pad11) -> /sec_counter/Q01234
- U25 pad 12: GND -> /sec_counter/Q0123
- U25 pad 13: GND -> /sec_counter/Q4
- U25 pad 8: unconnected-(U25-Pad8) -> /sec_counter/Q0123
- U25 pad 9: GND -> /sec_counter/Q012
- U28 pad 11: /min_counter/ones_D3 -> unconnected-(U28-Pad11)
- U28 pad 12: Net-(U28-Pad12) -> GND
- U28 pad 13: /min_counter/~{=9?} -> GND
- U29 pad 1: /A0 -> /A1
- U29 pad 10: /min_counter/~{=9?} -> /min_counter/~{tens_Q3}
- U29 pad 2: /B0 -> /min_counter/~{tens_Q1}
- U29 pad 3: /min_counter/ones_Q01 -> Net-(U29-Pad3)
- U29 pad 4: /min_counter/ones_Q01 -> Net-(U29-Pad3)
- U29 pad 5: /C0 -> Net-(U29-Pad5)
- U29 pad 6: /min_counter/ones_Q012 -> Net-(U29-Pad12)
- U29 pad 8: /min_counter/ones_D2 -> Net-(U29-Pad5)
- U29 pad 9: Net-(U29-Pad9) -> /C1
- U30 pad 6: Net-(U29-Pad9) -> Net-(U30-Pad6)
- U30 pad 8: Net-(U28-Pad12) -> Net-(U30-Pad8)
- U32 pad 10: /min_counter/~{tens_Q3} -> /min_counter/~{=9?}
- U32 pad 11: /min_counter/tens_Q012 -> /min_counter/ones_D3
- U32 pad 12: /min_counter/tens_Q01 -> Net-(U30-Pad8)
- U32 pad 13: /C1 -> /min_counter/~{=9?}
- U32 pad 8: Net-(U32-Pad8) -> /min_counter/ones_D2
- U32 pad 9: /C1 -> Net-(U30-Pad6)
- U33 pad 1: /A1 -> /A0
- U33 pad 11: /min_counter/tens_D3 -> /min_counter/tens_Q012
- U33 pad 12: Net-(U33-Pad12) -> /min_counter/tens_Q01
- U33 pad 13: /min_counter/~{=59?} -> /C1
- U33 pad 2: /min_counter/~{tens_Q1} -> /B0
- U33 pad 3: Net-(U33-Pad3) -> /min_counter/ones_Q01
- U33 pad 4: Net-(U33-Pad3) -> /min_counter/ones_Q01
- U33 pad 5: Net-(U32-Pad8) -> /C0
- U33 pad 6: Net-(U29-Pad12) -> /min_counter/ones_Q012
- U36 pad 8: Net-(U33-Pad12) -> Net-(U36-Pad8)
- U37 pad 11: unconnected-(U37-Pad11) -> /min_counter/tens_D3
- U37 pad 12: GND -> Net-(U36-Pad8)
- U37 pad 13: GND -> /min_counter/~{=59?}
- U42 pad 10: /hour_counter/~{=9 or =11?} -> /B3
- U42 pad 11: /hour_counter/ones_D3 -> /hour_counter/tens_Q012
- U42 pad 12: Net-(U39-Pad8) -> /hour_counter/tens_Q01
- U42 pad 13: /hour_counter/~{=9 or =11?} -> /C3
- U42 pad 8: /hour_counter/ones_D2 -> /hour_counter/tens_Q01
- U42 pad 9: Net-(U39-Pad6) -> /hour_counter/tens_Q0
- U43 pad 10: /B3 -> /hour_counter/~{=9 or =11?}
- U43 pad 11: /hour_counter/tens_Q012 -> /hour_counter/ones_D3
- U43 pad 12: /hour_counter/tens_Q01 -> Net-(U39-Pad8)
- U43 pad 13: /C3 -> /hour_counter/~{=9 or =11?}
- U43 pad 8: /hour_counter/tens_Q01 -> /hour_counter/ones_D2
- U43 pad 9: /hour_counter/tens_Q0 -> Net-(U39-Pad6)
- U47 pad 1: /A2 -> /hour_counter/~{tens_Q0}
- U47 pad 2: /hour_counter/~{ones_Q1} -> /hour_counter/~{=11?}
- U47 pad 3: Net-(U47-Pad3) -> /hour_counter/tens_D0
- U47 pad 4: /hour_counter/~{ones_Q2} -> Net-(U44-Pad3)
- U47 pad 5: /hour_counter/~{ones_Q3} -> /hour_counter/~{=11?}
- U47 pad 6: Net-(U47-Pad6) -> /hour_counter/tens_D1
- U48 pad 1: /hour_counter/~{tens_Q0} -> /A2
- U48 pad 10: Net-(U47-Pad6) -> Net-(U48-Pad10)
- U48 pad 2: /hour_counter/~{=11?} -> /hour_counter/~{ones_Q1}
- U48 pad 3: /hour_counter/tens_D0 -> Net-(U48-Pad3)
- U48 pad 4: Net-(U44-Pad3) -> /hour_counter/~{ones_Q2}
- U48 pad 5: /hour_counter/~{=11?} -> /hour_counter/~{ones_Q3}
- U48 pad 6: /hour_counter/tens_D1 -> Net-(U48-Pad10)
- U48 pad 9: Net-(U47-Pad3) -> Net-(U48-Pad3)
- U50 pad 10: GND -> Net-(U50-Pad10)
- U50 pad 11: Net-(U15-Pad9) -> unconnected-(U50-Pad11)
- U50 pad 12: Net-(U50-Pad12) -> GND
- U50 pad 13: Net-(U50-Pad13) -> GND
- U50 pad 3: Net-(U50-Pad13) -> Net-(U50-Pad10)
- U50 pad 6: Net-(U50-Pad12) -> Net-(U50-Pad6)
- U50 pad 8: unconnected-(U50-Pad8) -> Net-(U15-Pad9)
- U50 pad 9: GND -> Net-(U50-Pad6)
- U51 pad 10: /hour_counter/~{ones_Q1} -> Net-(U51-Pad10)
- U51 pad 11: Net-(U51-Pad11) -> unconnected-(U51-Pad11)
- U51 pad 12: /hour_counter/~{ones_Q2} -> GND
- U51 pad 13: /D2 -> GND
- U51 pad 6: Net-(U51-Pad6) -> Net-(U51-Pad10)
- U51 pad 8: Net-(U51-Pad8) -> /hour_counter/=1?
- U51 pad 9: /A2 -> Net-(U51-Pad3)
- U53 pad 1: Net-(U51-Pad3) -> /A2
- U53 pad 10: GND -> Net-(U53-Pad10)
- U53 pad 2: Net-(U51-Pad6) -> /hour_counter/~{ones_Q1}
- U53 pad 3: /hour_counter/=1? -> Net-(U53-Pad3)
- U53 pad 4: Net-(U51-Pad8) -> /hour_counter/~{ones_Q2}
- U53 pad 5: Net-(U51-Pad11) -> /D2
- U53 pad 6: /hour_counter/=9? -> Net-(U53-Pad10)
- U53 pad 8: unconnected-(U53-Pad8) -> /hour_counter/=9?
- U53 pad 9: GND -> Net-(U53-Pad3)
Routing:
- net /CLK_1sec: track 0.00 -> 218.8 mm
- net Net-(D2-Pad1): track 0.00 -> 207.8 mm
- net Net-(D1-Pad1): track 0.00 -> 101.5 mm, vias 0 -> 2
- net /AM/PM: track 0.00 -> 85.5 mm, vias 0 -> 2
- net /RESET_STATE: track 0.00 -> 66.7 mm
- net /sec_counter/D5: track 0.00 -> 59.6 mm
- net Net-(R21-Pad2): track 0.00 -> 56.5 mm
- net Net-(R22-Pad2): track 0.00 -> 56.2 mm
- net Net-(R1-Pad1): track 0.00 -> 54.2 mm
- net Net-(R19-Pad2): track 0.00 -> 53.4 mm
- net /sec_counter/Q3: track 0.00 -> 52.9 mm
- net Net-(R3-Pad1): track 0.00 -> 52.6 mm
- net Net-(R20-Pad2): track 0.00 -> 49.0 mm
- net Net-(R28-Pad2): track 0.00 -> 47.9 mm
- net Net-(R29-Pad2): track 0.00 -> 46.5 mm
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Other:
- board text added: "PM"
- board text added: "SET TIME"

Commit message: started routing
Connections:
- U4 pad 1: /+MIN BUTTON -> /+MIN
- U4 pad 4: /+HOUR BUTTON -> /+HOUR
Routing:
- net /B0: track 0.00 -> 236.2 mm, vias 0 -> 8
- net /A0: track 0.00 -> 228.5 mm, vias 0 -> 10
- net /A1: track 0.00 -> 222.2 mm, vias 0 -> 6
- net /~{RESET_PULSE}: track 5.76 -> 220.7 mm, vias 0 -> 4
- net /C0: track 0.00 -> 214.4 mm, vias 0 -> 5
- net /C1: track 0.00 -> 198.6 mm, vias 0 -> 6
- net /B1: track 0.00 -> 184.8 mm, vias 0 -> 4
- net /D0: track 0.00 -> 184.1 mm, vias 0 -> 4
- net /D1: track 0.00 -> 149.6 mm, vias 0 -> 5
- net /min_counter/CLK_1min: track 0.00 -> 126.0 mm, vias 0 -> 2
- net /min_counter/=9?: track 0.00 -> 122.5 mm, vias 0 -> 3
- net /B3: track 0.00 -> 121.9 mm, vias 0 -> 4
- net /sec_counter/Q1: track 0.00 -> 120.1 mm, vias 0 -> 2
- net /min_counter/~{=59?}: track 0.00 -> 114.5 mm, vias 0 -> 6
- net /min_counter/=59?: track 0.00 -> 106.1 mm, vias 0 -> 1
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